File: MagicDeskCartDual.kicad_pcb (KiCad board)
At the start: 2 copper layers, 58.4 x 86.2 mm, 10 parts, among them U1 74LS174, U2 74LS02, U3 27C020, U4 C64-Exp-Port, U5 C64-Exp-Port

Commit message: Tuning layout.
Other:
- outline, holes or cut-outs redrawn
- board text added: "MagicDeskCart Dual"
- board text added: "Rev.1"

Commit message: Tuning layout.
Parts:
- added G***: LOGO, Logo:bigby2, F.Cu at (88.5, 76.7)

Commit message: Tuning layout.
Other:
- board text added: "https://github.com/hackup/MagicDeskDual"
Changed lines of the file:
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@@
   (general
     (thickness 1.6)
-    (drawings 14)
+    (drawings 15)
     (tracks 652)
     (zones 0)
@@
     )
   )
+  (gr_text https://github.com/hackup/MagicDeskDual (at 81.026 99.949 90) (layer B.SilkS)
+    (effects (font (size 1 1) (thickness 0.15)) (justify mirror))
+  )
   (gr_text Rev.1 (at 81.153 84.709 90) (layer F.SilkS)
